File: envelope_v1/envelope_v1.kicad_pcb (KiCad board)
At the start: 2 copper layers, 90 x 100 mm, 113 parts, among them J1 Conn_02x05_Odd_Even, J10 Conn_01x10, J2 Gate_A, J3 Trigger_A, J4 Attack_IN, J5 ENV_A, J6 Decay_IN, J7 Sustain_IN, J8 Release_IN, J9 Conn_01x10, Q1 2N3906, SW1 Gate_SW, SW2 Trig_SW, U1 TL074, U2 TL074, U3 AS3310

Commit message: Geographic re-annotate
Parts:
- renumbered C2 to C1, C13 to C10, C10 to C11, C3 to C12, C1 to C13, C4 to C2, C12 to C3, C9 to C4, C8 to C5, C5 to C6, C6 to C7, C11 to C8, C7 to C9, CALT_8 to CALT_1, CALT_5 to CALT_2, D2 to D10, D6 to D11, D5 to D2, D8 to D3, D9 to D4, D10 to D5, D11 to D6, D3 to D8, D4 to D9, H6 to H1, H3 to H2, H5 to H3, H2 to H4, H4 to H5, H1 to H6, J10 to J1, J9 to J10, J4 to J2, J6 to J3, J7 to J4, J8 to J5, J2 to J6, J3 to J7, J5 to J8, J1 to J9, R33 to R1, R22 to R10, R12 to R11, R11 to R12, R18 to R13, R21 to R14, R10 to R15, R29 to R16, R38 to R17, R53 to R18, R43 to R19, R30 to R2, R54 to R20, R27 to R21, R28 to R22, R42 to R23, R55 to R24, R56 to R25, R52 to R26, R44 to R27, R39 to R28, R51 to R29, R5 to R3, R48 to R30, R17 to R31, R16 to R32, R1 to R33, R3 to R34, R25 to R35, R15 to R36, R26 to R37, R24 to R38, R6 to R39, R9 to R40, R2 to R41, R8 to R42, R37 to R43, R36 to R44, R19 to R45, R31 to R46, R35 to R47, R47 to R48, R40 to R49, R34 to R5, R46 to R50, R45 to R51, R49 to R52, R13 to R53, R7 to R54, R23 to R55, R14 to R56, R41 to R6, R50 to R7, R20 to R8, R32 to R9, U3 to U2, U2 to U3
Connections:
- R_Attack1 pad MP: (no net) -> GND
- R_Decay1 pad MP: (no net) -> GND
- R_Release1 pad MP: (no net) -> GND
- R_Sustain1 pad MP: (no net) -> GND

Commit message: Cleanup and labels
Parts:
- renumbered CALT_1 to CALT_5, CALT_2 to CALT_6
Routing:
- net +12V: track 301.0 -> 304.3 mm, vias 10 -> 12
Other:
- board text added: "AS3310"
- board text added: "ATTACK"
- board text added: "DECAY"
- board text added: "ENV"
- board text added: "GATE"
- board text added: "RELEASE"
- board text added: "SUSTAIN"
- board text added: "TL074"
- board text added: "TRIG"
Changed lines of the file:
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@@
   (paper "A4")
   (title_block
-    (title "Envelope AS3310 ADSR")
+    (title "Envelope Generator AS3310")
     (date "2022-12-06")
     (rev "1.0")
@@
     (property "Sheetname" "")
     (attr through_hole)
-    (fp_text reference "CALT_1" (at 2.3 -2.9 90) (layer "B.SilkS")
+    (fp_text reference "CALT_5" (at 2.3 -2.9 90) (layer "B.SilkS")
       (effects (font (size 1 1) (thickness 0.15)) (justify mirror))
     )
@@
     (property "Sheetname" "")
     (attr through_hole)
-    (fp_text reference "CALT_2" (at 2.4 -2.9 90) (layer "B.SilkS")
+    (fp_text reference "CALT_6" (at 2.4 -2.9 90) (layer "B.SilkS")
       (effects (font (size 1 1) (thickness 0.15)) (justify mirror))
     )
@@
     )
   )
+  (gr_line (start 218.109944 113.5) (end 220.609944 113.5) (layer "B.SilkS") (width 0.15))
+  (gr_arc (start 222.609944 111) (mid 224.5 113.265966) (end 225.609944 116) (layer "B.SilkS") (width 0.15))
+  (gr_arc (start 222.609944 111) (mid 222.095649 112.638564) (end 220.609944 113.5) (layer "B.SilkS") (width 0.15))
+  (gr_arc (start 218.109944 113.5) (mid 217.17529 115.065346) (end 215.609944 116) (layer "B.SilkS") (width 0.15))
   (gr_line locked (start 145.25 145) (end 182.2 145) (layer "Dwgs.User") (width 0.15))
   (gr_line locked (start 145.25 133) (end 183 133) (layer "Dwgs.User") (width 0.15))
@@
   (gr_rect locked (start 190 50) (end 230 150) (layer "Edge.Cuts") (width 0.1) (fill none))
   (gr_rect locked (start 140 50) (end 180 150) (layer "Edge.Cuts") (width 0.1) (fill none))
+  (gr_text "ATTACK" (at 146.1 131) (layer "B.SilkS")
+    (effects (font (size 1 1) (thickness 0.15)) (justify mirror))
+  )
+  (gr_text "TRIG" (at 156 142.8) (layer "B.SilkS")
+    (effects (font (size 1 1) (thickness 0.15)) (justify mirror))
+  )
   (gr_text "v1.0 Nov 2022" (at 220.7 123.6) (layer "B.SilkS")
     (effects (font (size 1 1) (thickness 0.15)) (justify mirror))
   )
+  (gr_text "DECAY" (at 155.9 130.8) (layer "B.SilkS")
+    (effects (font (size 1 1) (thickness 0.15)) (justify mirror))
+  )
   (gr_text "PCB B" (at 176.8 51.6) (layer "B.SilkS")
     (effects (font (size 1 1) (thickness 0.15)) (justify mirror))
   )
+  (gr_text "SUSTAIN" (at 165.8 130.9) (layer "B.SilkS")
+    (effects (font (size 1 1) (thickness 0.15)) (justify mirror))
+  )
+  (gr_text "ENV" (at 178.8 140.4 90) (layer "B.SilkS")
+    (effects (font (size 1 1) (thickness 0.15)) (justify mirror))
+  )
   (gr_text "AS3310 ADSR" (at 220.7 121.599999) (layer "B.SilkS")
     (effects (font (size 1 1) (thickness 0.15)) (justify mirror))
   )
+  (gr_text "TL074" (at 210 89.9) (layer "B.SilkS")
+    (effects (font (size 1 1) (thickness 0.15)) (justify mirror))
+  )
   (gr_text "RobotDialogs\n" (at 220.7 117.6) (layer "B.SilkS")
     (effects (font (size 1 1) (thickness 0.15)) (justify mirror))
@@
     (effects (font (size 1 1) (thickness 0.15)) (justify mirror))
   )
+  (gr_text "GATE" (at 146.1 143) (layer "B.SilkS")
+    (effects (font (size 1 1) (thickness 0.15)) (justify mirror))
+  )
+  (gr_text "TL074" (at 210 144.9) (layer "B.SilkS")
+    (effects (font (size 1 1) (thickness 0.15)) (justify mirror))
+  )
+  (gr_text "RELEASE" (at 175.6 131) (layer "B.SilkS")
+    (effects (font (size 1 1) (thickness 0.15)) (justify mirror))
+  )
   (gr_text "Envelope Generator" (at 220.7 119.6) (layer "B.SilkS")
     (effects (font (size 1 1) (thickness 0.15)) (justify mirror))
   )
+  (gr_text "AS3310" (at 209.9 116.2) (layer "B.SilkS")
+    (effects (font (size 1 1) (thickness 0.15)) (justify mirror))
+  )
   (gr_text "Envelope Generator" (at 155 54) (layer "F.SilkS")
     (effects (font (size 1 1) (thickness 0.15)))
@@
   (segment (start 211.3 80.0375) (end 213.7575 80.0375) (width 0.6) (layer "F.Cu") (net 1))
   (segment (start 214.1575 134.6375) (end 213.8 134.995) (width 0.6) (layer "F.Cu") (net 1))
+  (segment (start 221.6 118.6) (end 221.6 119.7) (width 0.6) (layer "F.Cu") (net 1))
   (segment (start 146.7 100.9) (end 147.8 99.8) (width 0.6) (layer "F.Cu") (net 1))
   (segment (start 206.1425 108.8375) (end 206.18 108.8) (width 0.6) (layer "F.Cu") (net 1))
@@
   (segment (start 217 136) (end 221.6 136) (width 0.6) (layer "F.Cu") (net 1))
   (segment (start 216.8 134.6375) (end 214.1575 134.6375) (width 0.6) (layer "F.Cu") (net 1))
+  (segment (start 203.56 118.64) (end 203.56 116.36) (width 0.6) (layer "F.Cu") (net 1))
   (segment (start 150 87) (end 147.840489 84.840489) (width 0.6) (layer "F.Cu") (net 1))
   (segment (start 147.8 89.2) (end 150 87) (width 0.6) (layer "F.Cu") (net 1))
   (via (at 203.56 116.36) (size 0.7) (drill 0.4) (layers "F.Cu" "B.Cu") (net 1))
+  (via (at 221.6 119.7) (size 0.7) (drill 0.4) (layers "F.Cu" "B.Cu") (net 1))
   (via (at 223 67.7) (size 0.7) (drill 0.4) (layers "F.Cu" "B.Cu") (net 1))
   (via (at 161.5 121) (size 0.7) (drill 0.4) (layers "F.Cu" "B.Cu") (net 1))
@@
   (via (at 203.56 118.64) (size 0.7) (drill 0.4) (layers "F.Cu" "B.Cu") (net 1))
   (via (at 221.6 136) (size 0.7) (drill 0.4) (layers "F.Cu" "B.Cu") (net 1))
+  (via (at 203.56 117.46) (size 0.7) (drill 0.4) (layers "F.Cu" "B.Cu") (net 1))
   (via (at 146.7 115.2) (size 0.7) (drill 0.4) (layers "F.Cu" "B.Cu") (net 1))
   (via (at 221.6 118.6) (size 0.7) (drill 0.4) (layers "F.Cu" "B.Cu") (net 1))
@@
   (segment (start 146.7 114.2) (end 146.7 115.2) (width 0.6) (layer "B.Cu") (net 1))
   (segment (start 203.56 122.76) (end 203.9 123.1) (width 0.6) (layer "B.Cu") (net 1))
+  (segment (start 203.56 116.36) (end 203.56 117.46) (width 0.6) (layer "B.Cu") (net 1))
   (segment (start 223.2 71.5) (end 223.2 67.9) (width 0.6) (layer "B.Cu") (net 1))
   (segment (start 223.2 67.9) (end 223 67.7) (width 0.6) (layer "B.Cu") (net 1))
   (segment (start 146.665 116.435) (end 146.665 115.235) (width 0.6) (layer "B.Cu") (net 1))
-  (segment (start 203.56 116.36) (end 203.56 118.64) (width 0.6) (layer "B.Cu") (net 1))
-  (segment (start 221.6 136) (end 221.6 118.6) (width 0.6) (layer "B.Cu") (net 1))
   (segment (start 203.56 108.84) (end 203.56 116.36) (width 0.6) (layer "B.Cu") (net 1))
   (segment (start 161.5 121) (end 159.5 121) (width 0.6) (layer "B.Cu") (net 1))
   (segment (start 206.18 108.8) (end 203.6 108.8) (width 0.6) (layer "B.Cu") (net 1))
   (segment (start 159.5 117.67) (end 158.265 116.435) (width 0.6) (layer "B.Cu") (net 1))
+  (segment (start 221.6 119.7) (end 221.6 103.7) (width 0.6) (layer "B.Cu") (net 1))
   (segment (start 203.56 118.64) (end 203.56 122.76) (width 0.6) (layer "B.Cu") (net 1))
   (segment (start 220.6 87.1) (end 220.6 80) (width 0.6) (layer "B.Cu") (net 1))
   (segment (start 146.665 115.235) (end 146.7 115.2) (width 0.6) (layer "B.Cu") (net 1))
+  (segment (start 203.56 117.46) (end 203.56 118.64) (width 0.6) (layer "B.Cu") (net 1))
   (segment (start 146.665 116.435) (end 158.265 116.435) (width 0.6) (layer "B.Cu") (net 1))
   (segment (start 163.45 65) (end 152 65) (width 0.6) (layer "B.Cu") (net 1))
@@
   (segment (start 220.6 80) (end 220.6 74.1) (width 0.6) (layer "B.Cu") (net 1))
   (segment (start 163.45 69.8) (end 163.45 65) (width 0.6) (layer "B.Cu") (net 1))
-  (segment (start 221.6 118.6) (end 221.6 103.7) (width 0.6) (layer "B.Cu") (net 1))
+  (segment (start 221.6 136) (end 221.6 119.7) (width 0.6) (layer "B.Cu") (net 1))
   (segment (start 206.7975 76.8375) (end 206.18 77.455) (width 0.6) (layer "F.Cu") (net 2))
   (segment (start 208.8 76.8375) (end 206.7975 76.8375) (width 0.6) (layer "F.Cu") (net 2))
@@
   (segment (start 219.3 142.85) (end 216.8 142.85) (width 0.6) (layer "F.Cu") (net 52))
   (segment (start 223.1 139.5) (end 219.55 139.5) (width 0.6) (layer "F.Cu") (net 53))
-  (segment (start 206.18 113.88) (end 208.2 115.9) (width 0.6) (layer "F.Cu") (net 53))
-  (segment (start 208.20048 115.90048) (end 223.09952 115.90048) (width 0.6) (layer "F.Cu") (net 53))
-  (segment (start 223.09952 115.90048) (end 223.1 115.9) (width 0.6) (layer "F.Cu") (net 53))
-  (segment (start 208.2 115.9) (end 208.20048 115.90048) (width 0.6) (layer "F.Cu") (net 53))
+  (segment (start 222.6 115.4) (end 223.1 115.9) (width 0.6) (layer "F.Cu") (net 53))
+  (segment (start 207.7 115.4) (end 222.6 115.4) (width 0.6) (layer "F.Cu") (net 53))
+  (segment (start 206.18 113.88) (end 207.7 115.4) (width 0.6) (layer "F.Cu") (net 53))
   (segment (start 219.55 139.5) (end 219.3 139.75) (width 0.6) (layer "F.Cu") (net 53))
   (via (at 223.1 115.9) (size 0.7) (drill 0.4) (layers "F.Cu" "B.Cu") (net 53))
@@
     )
   )
+  (group "" (id 0af0432e-dc19-402a-9bf6-17313aa4158f)
+    (members
+      31a66d8b-f987-45ba-899e-0699a385af59
+      5946fd19-6935-440f-842e-41314253fabe
+      6b725547-9a1c-4d08-a1ce-a2c9b1828e82
+      c1400dad-c8b4-4b68-bd23-d8f70924358c
+    )
+  )

Commit message: v1.1 fixes
Parts:
- moved D6 2.54 mm to (145.0, 111.4)
- moved R52 2.54 mm to (156.4, 111.4)
Connections:
- J10 pad 8: TO_OUT -> FROM_REL
- J10 pad 9: FROM_REL -> TO_OUT
Routing:
- net TO_OUT: track 61.6 -> 58.3 mm
- net Net-(J5-PadT): track 42.5 -> 41.4 mm, vias 1 -> 0
Other:
- board text added: "v1.1 Jan 2023"
- board text removed: "v1.0 Nov 2022"
