File: envelope_v1/envelope_v1.kicad_sch (KiCad schematic)
At the start: 113 parts, among them J1 Conn_02x05_Odd_Even, J10 Conn_01x10, J2 Gate_A, J3 Trigger_A, J4 Attack_IN, J5 ENV_A, J6 Decay_IN, J7 Sustain_IN, J8 Release_IN, J9 Conn_01x10, Q1 2N3906, SW1 Gate_SW, SW2 Trig_SW, U1 TL074, U2 TL074, U3 AS3310

Commit message: Geographic re-annotate
Parts:
- R_Attack1, R_Decay1, R_Release1, R_Sustain1: symbol Device:R_Potentiometer -> Device:R_Potentiometer_MountingPin
- renumbered C2 to C1, C13 to C10, C10 to C11, C3 to C12, C1 to C13, C4 to C2, C12 to C3, C9 to C4, C8 to C5, C5 to C6, C6 to C7, C11 to C8, C7 to C9, CALT_8 to CALT_1, CALT_5 to CALT_2, D2 to D10, D6 to D11, D5 to D2, D8 to D3, D9 to D4, D10 to D5, D11 to D6, D3 to D8, D4 to D9, H6 to H1, H3 to H2, H5 to H3, H2 to H4, H4 to H5, H1 to H6, J10 to J1, J9 to J10, J4 to J2, J6 to J3, J7 to J4, J8 to J5, J2 to J6, J3 to J7, J5 to J8, J1 to J9, R33 to R1, R22 to R10, R12 to R11, R11 to R12, R18 to R13, R21 to R14, R10 to R15, R29 to R16, R38 to R17, R53 to R18, R43 to R19, R30 to R2, R54 to R20, R27 to R21, R28 to R22, R42 to R23, R55 to R24, R56 to R25, R52 to R26, R44 to R27, R39 to R28, R51 to R29, R5 to R3, R48 to R30, R17 to R31, R16 to R32, R1 to R33, R3 to R34, R25 to R35, R15 to R36, R26 to R37, R24 to R38, R6 to R39, R9 to R40, R2 to R41, R8 to R42, R37 to R43, R36 to R44, R19 to R45, R31 to R46, R35 to R47, R47 to R48, R40 to R49, R34 to R5, R46 to R50, R45 to R51, R49 to R52, R13 to R53, R7 to R54, R23 to R55, R14 to R56, R41 to R6, R50 to R7, R20 to R8, R32 to R9, U3 to U2, U2 to U3
Connections:
- net GND: now also R_Attack1.MP (MountPin), R_Decay1.MP (MountPin), R_Release1.MP (MountPin), R_Sustain1.MP (MountPin)

Commit message: Cleanup and labels
Parts:
- renumbered CALT_1 to CALT_5, CALT_2 to CALT_6
Other:
- title: Envelope AS3310 ADSR -> Envelope Generator AS3310
Changed lines of the file:
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@@
   (paper "A4")
   (title_block
-    (title "Envelope AS3310 ADSR")
+    (title "Envelope Generator AS3310")
     (date "2022-12-06")
     (rev "1.0")
@@
   (symbol (lib_id "Device:C") (at 163.83 60.325 90) (unit 1)
     (in_bom yes) (on_board yes)
-    (property "Reference" "CALT_2" (id 0) (at 161.29 59.055 0)
+    (property "Reference" "CALT_6" (id 0) (at 161.29 59.055 0)
       (effects (font (size 1.27 1.27)) (justify left))
     )
@@
   (symbol (lib_id "Device:C") (at 173.355 128.27 0) (unit 1)
     (in_bom yes) (on_board yes)
-    (property "Reference" "CALT_1" (id 0) (at 174.625 125.73 0)
+    (property "Reference" "CALT_5" (id 0) (at 174.625 125.73 0)
       (effects (font (size 1.27 1.27)) (justify left))
     )
@@
     )
     (path "/43968b13-86a1-43f9-a397-25296aa1c52a"
-      (reference "CALT_1") (unit 1) (value "39nF") (footprint "Capacitor_THT:C_Disc_D5.1mm_W3.2mm_P5.00mm")
+      (reference "CALT_5") (unit 1) (value "39nF") (footprint "Capacitor_THT:C_Disc_D5.1mm_W3.2mm_P5.00mm")
     )
     (path "/2d00b297-b75e-4ac2-8956-5cdf76e11101"
-      (reference "CALT_2") (unit 1) (value "1uF") (footprint "Capacitor_THT:C_Disc_D5.1mm_W3.2mm_P5.00mm")
+      (reference "CALT_6") (unit 1) (value "1uF") (footprint "Capacitor_THT:C_Disc_D5.1mm_W3.2mm_P5.00mm")
     )
     (path "/776694d1-8de6-4198-adee-6b625f1fbdb9"

Commit message: v1.1 fixes
Connections:
- net FROM_REL: now also J10.8 (Pin_8); no longer J10.9 (Pin_9)
- net TO_OUT: now also J10.9 (Pin_9); no longer J10.8 (Pin_8)
